Commit message: Gazebo world fixed

File: src/puma560_description/urdf/puma560_robot.urdf (robot description, URDF)
Before this commit: robot Puma560, 8 links, 7 joints
Links:
- removed link world
- added link base_link
Joints:
- removed joint dummy_joint
- added joint base_link_joint: type fixed, parent base_link, origin xyz=0 0 0 rpy=0 0 0

Commit message: Updated URDF, not spawning anymore

File: src/puma560_description/urdf/puma560_robot.urdf (robot description, URDF)
Before this commit: robot Puma560, 8 links, 7 joints
Links:
- link link1: geometry collision mesh filename=package://puma560_description/meshes/puma_link1.stl; visual mesh filename=package://puma560_description/meshes/puma_link1.stl
- link link2: mass 0.5 -> 17.4; geometry collision mesh filename=package://puma560_description/meshes/puma_link2.stl; visual mesh filename=package://puma560_description/meshes/puma_link2.stl
- link link3: mass 0.5 -> 4.8; geometry collision mesh filename=package://puma560_description/meshes/puma_link3.stl; visual mesh filename=package://puma560_description/meshes/puma_link3.stl
- link link4: mass 0.5 -> 0.82; geometry collision mesh filename=package://puma560_description/meshes/puma_link4.stl; visual mesh filename=package://puma560_description/meshes/puma_link4.stl
- link link5: mass 0.5 -> 0.34; geometry collision mesh filename=package://puma560_description/meshes/puma_link5.stl; visual mesh filename=package://puma560_description/meshes/puma_link5.stl
- link link6: mass 0.5 -> 0.09; geometry collision mesh filename=package://puma560_description/meshes/puma_link6.stl; visual mesh filename=package://puma560_description/meshes/puma_link6.stl
- link link7: mass 0.5 -> 2.24; geometry collision mesh filename=package://puma560_description/meshes/puma_link7.stl; visual mesh filename=package://puma560_description/meshes/puma_link7.stl

Commit message: Problem fixed, strange inertias added

File: src/puma560_description/urdf/puma560_robot.urdf (robot description, URDF)
Before this commit: robot Puma560, 8 links, 7 joints
Links:
- removed link base_link
- added link world
- link link1: geometry collision mesh filename=package://puma560_description/meshes/puma_link1.stl scale=0.0254 0.0254 0.0254; visual mesh filename=package://puma560_description/meshes/puma_link1.stl scale=0.0254 0.0254 0.0254
- link link2: geometry collision mesh filename=package://puma560_description/meshes/puma_link2.stl scale=0.0254 0.0254 0.0254; visual mesh filename=package://puma560_description/meshes/puma_link2.stl scale=0.0254 0.0254 0.0254
- link link3: geometry collision mesh filename=package://puma560_description/meshes/puma_link3.stl scale=0.0254 0.0254 0.0254; visual mesh filename=package://puma560_description/meshes/puma_link3.stl scale=0.0254 0.0254 0.0254
- link link4: geometry collision mesh filename=package://puma560_description/meshes/puma_link4.stl scale=0.0254 0.0254 0.0254; visual mesh filename=package://puma560_description/meshes/puma_link4.stl scale=0.0254 0.0254 0.0254
- link link5: geometry collision mesh filename=package://puma560_description/meshes/puma_link5.stl scale=0.0254 0.0254 0.0254; visual mesh filename=package://puma560_description/meshes/puma_link5.stl scale=0.0254 0.0254 0.0254
- link link6: geometry collision mesh filename=package://puma560_description/meshes/puma_link6.stl scale=0.0254 0.0254 0.0254; visual mesh filename=package://puma560_description/meshes/puma_link6.stl scale=0.0254 0.0254 0.0254
- link link7: geometry collision mesh filename=package://puma560_description/meshes/puma_link7.stl scale=0.0254 0.0254 0.0254; visual mesh filename=package://puma560_description/meshes/puma_link7.stl scale=0.0254 0.0254 0.0254
Joints:
- removed joint base_link_joint
- added joint dummy_joint: type fixed, parent world, child link1

Commit message: Controller connected

File: src/puma560_description/urdf/puma560_robot.urdf (robot description, URDF)
Before this commit: robot Puma560, 8 links, 7 joints
Joints:
- removed joint j1
- removed joint j2
- removed joint j3
- removed joint j4
- removed joint j5
- removed joint j6
- added joint effector_revolute: type revolute, parent link6, child link7, origin xyz=0 0.0558 0 rpy=-1.570796325 0 0, axis 0 0 1, limit lower=-1.570796325 upper=1.570796325 effort=1000.0 velocity=0
- added joint elbow: type revolute, parent link3, child link4, origin xyz=0.4318 -0.0203 0.1501 rpy=0 0 -1.570796325, axis 0 0 1, limit lower=-1.570796325 upper=1.570796325 effort=1000.0 velocity=0
- added joint platform: type revolute, parent link1, child link2, origin xyz=0 0 0.6718 rpy=1.570796325 0 0, axis 0 1 0, limit lower=-3.14159265 upper=3.14159265 effort=1000.0 velocity=0
- added joint shoulder: type revolute, parent link2, child link3, origin xyz=0 0 0 rpy=0 0 1.570796325, axis 0 0 1, limit lower=-1.570796325 upper=1.570796325 effort=1000.0 velocity=0
- added joint wrist_bend: type revolute, parent link5, child link6, origin xyz=0 0 0.4331 rpy=1.570796325 0 0, axis 0 0 1, limit lower=-1.570796325 upper=1.570796325 effort=1000.0 velocity=0
- added joint wrist_revolute: type revolute, parent link4, child link5, origin xyz=0 0 0 rpy=1.570796325 0 1.570796325, axis 0 0 1, limit lower=-1.570796325 upper=1.570796325 effort=1000.0 velocity=0

Commit message: Optimizer test added. Position set plugin added. Joints enumeration check added

File: src/puma560_description/urdf/puma560_robot.urdf (robot description, URDF)
Before this commit: robot Puma560, 8 links, 7 joints
Joints:
- joint effector_revolute: limit lower=-1.570796325 upper=1.570796325 effort=1000.0 velocity=0 -> lower=-1.570796325 upper=1.570796325 effort=21.3 velocity=100
- joint elbow: limit lower=-1.570796325 upper=1.570796325 effort=1000.0 velocity=0 -> lower=-1.570796325 upper=1.570796325 effort=89.4 velocity=100
- joint platform: limit lower=-3.14159265 upper=3.14159265 effort=1000.0 velocity=0 -> lower=-3.14159265 upper=3.14159265 effort=97.6 velocity=100
- joint shoulder: limit lower=-1.570796325 upper=1.570796325 effort=1000.0 velocity=0 -> lower=-1.570796325 upper=1.570796325 effort=186.4 velocity=100
- joint wrist_bend: limit lower=-1.570796325 upper=1.570796325 effort=1000.0 velocity=0 -> lower=-1.570796325 upper=1.570796325 effort=20.1 velocity=100
- joint wrist_revolute: limit lower=-1.570796325 upper=1.570796325 effort=1000.0 velocity=0 -> lower=-1.570796325 upper=1.570796325 effort=24.2 velocity=100
