Commit message: Robots lag every time. Not enough time to mess with this anymore

File: src/puma560_description/xacro/puma560_robot.xacro (robot description, xacro)
@@ -1,7 +1,3 @@
 <?xml version="1.0" ?>
-<!-- =================================================================================== -->
-<!-- |    This document was autogenerated by xacro from puma560_robot.urdf.xacro       | -->
-<!-- |    EDITING THIS FILE BY HAND IS NOT RECOMMENDED                                 | -->
-<!-- =================================================================================== -->
 <robot name="Puma560" xmlns:xacro="http://www.ros.org/wiki/xacro">
   <material name="blue">
@@ -17,12 +13,12 @@
   <link name="world">
   </link>
-  <joint name="dummy_joint" type="fixed">
+  <joint name="$(arg robot_name)_dummy_joint" type="fixed">
         <parent link="world"/>
-        <child link="link1"/>
-  </joint>
-  <link name="link1">
+        <child link="$(arg robot_name)_link1"/>
+  </joint>
+  <link name="$(arg robot_name)_link1">
     <inertial>
             <mass value="0.5"/>
-            <origin rpy="0 0 0" xyz="0 0 0"/>
+            <origin rpy="0 0 0" xyz="$(arg pos_x) $(arg pos_y) 0.0"/>
             <inertia ixx="0" ixy="0" ixz="0" iyy="0" iyz="0" izz="0.35"/>
     </inertial>
@@ -36,10 +32,10 @@
     <collision>
       <geometry>
-        <mesh filename="package://puma560_description/meshes/puma_link1.stl" scale="0.0254 0.0254 0.0254"/>
+        <box size="0.01 0.01 0.01"/>
       </geometry>
       <origin rpy="0 0 1.570796325"/>
     </collision>
   </link>
-  <link name="link2">
+  <link name="$(arg robot_name)_link2">
   <inertial>
           <mass value="17.4"/>
@@ -56,12 +52,12 @@
     <collision>
       <geometry>
-        <mesh filename="package://puma560_description/meshes/puma_link2.stl" scale="0.0254 0.0254 0.0254"/>
+        <box size="0.01 0.01 0.01"/>
       </geometry>
       <origin rpy="0 0 0" xyz="0 0 -0.1"/>
     </collision>
   </link>
-  <joint name="platform" type="revolute">
-    <parent link="link1"/>
-    <child link="link2"/>
+  <joint name="$(arg robot_name)_platform" type="revolute">
+    <parent link="$(arg robot_name)_link1"/>
+    <child link="$(arg robot_name)_link2"/>
     <origin rpy="1.570796325 0 0" xyz="0 0 0.6718"/>
     <axis xyz="0 1 0"/>
@@ -69,5 +65,5 @@
     <limit effort="97.6" lower="-3.14159265" upper="3.14159265" velocity="100"/>
   </joint>
-  <link name="link3">
+  <link name="$(arg robot_name)_link3">
   <inertial>
           <mass value="4.8"/>
@@ -84,12 +80,12 @@
      <collision>
       <geometry>
-        <mesh filename="package://puma560_description/meshes/puma_link3.stl" scale="0.0254 0.0254 0.0254"/>
+        <box size="0.01 0.01 0.01"/>
       </geometry>
       <origin xyz="0 0 0.1936"/>
     </collision>
   </link>
-  <joint name="shoulder" type="revolute">
-    <parent link="link2"/>
-    <child link="link3"/>
+  <joint name="$(arg robot_name)_shoulder" type="revolute">
+    <parent link="$(arg robot_name)_link2"/>
+    <child link="$(arg robot_name)_link3"/>
     <origin rpy="0 0 1.570796325" xyz="0 0 0"/>
     <axis xyz="0 0 1"/>
@@ -97,5 +93,5 @@
     <limit effort="186.4" lower="-1.570796325" upper="1.570796325" velocity="100"/>
   </joint>
-  <link name="link4">
+  <link name="$(arg robot_name)_link4">
   <inertial>
           <mass value="0.82"/>
@@ -112,12 +108,12 @@
     <collision>
       <geometry>
-        <mesh filename="package://puma560_description/meshes/puma_link4.stl" scale="0.0254 0.0254 0.0254"/>
+        <box size="0.01 0.01 0.01"/>
       </geometry>
       <origin rpy="0 0 0" xyz="0 0 0"/>
     </collision>
   </link>
-  <joint name="elbow" type="revolute">
-    <parent link="link3"/>
-    <child link="link4"/>
+  <joint name="$(arg robot_name)_elbow" type="revolute">
+    <parent link="$(arg robot_name)_link3"/>
+    <child link="$(arg robot_name)_link4"/>
     <origin rpy="0 0 -1.570796325" xyz="0.4318 -0.0203 0.1501"/>
     <axis xyz="0 0 1"/>
@@ -125,5 +121,5 @@
     <limit effort="89.4" lower="-1.570796325" upper="1.570796325" velocity="100"/>
   </joint>
-  <link name="link5">
+  <link name="$(arg robot_name)_link5">
   <inertial>
     <mass value="0.34"/>
@@ -140,17 +136,17 @@
     <collision>
       <geometry>
-        <mesh filename="package://puma560_description/meshes/puma_link5.stl" scale="0.0254 0.0254 0.0254"/>
+        <box size="0.01 0.01 0.01"/>
       </geometry>
       <origin rpy="0 0 1.570796325" xyz="0 0 0.3621"/>
     </collision>
   </link>
-  <joint name="wrist_revolute" type="revolute">
-    <parent link="link4"/>
-    <child link="link5"/>
+  <joint name="$(arg robot_name)_wrist_revolute" type="revolute">
+    <parent link="$(arg robot_name)_link4"/>
+    <child link="$(arg robot_name)_link5"/>
     <origin rpy="1.570796325 0 1.570796325" xyz="0 0 0"/>
     <axis xyz="0 0 1"/>
     <limit effort="24.2" lower="-1.570796325" upper="1.570796325" velocity="100"/>
   </joint>
-  <link name="link6">
+  <link name="$(arg robot_name)_link6">
   <inertial>
           <mass value="0.09"/>
@@ -167,17 +163,17 @@
     <collision>
       <geometry>
-        <mesh filename="package://puma560_description/meshes/puma_link6.stl" scale="0.0254 0.0254 0.0254"/>
+        <box size="0.01 0.01 0.01"/>
       </geometry>
       <origin rpy="3.14159265 0 1.570796325" xyz="0 0 0"/>
     </collision>
   </link>
-  <joint name="wrist_bend" type="revolute">
-    <parent link="link5"/>
-    <child link="link6"/>
+  <joint name="$(arg robot_name)_wrist_bend" type="revolute">
+    <parent link="$(arg robot_name)_link5"/>
+    <child link="$(arg robot_name)_link6"/>
     <origin rpy="1.570796325 0 0" xyz="0 0 0.4331"/>
     <axis xyz="0 0 1"/>
     <limit effort="20.1" lower="-1.570796325" upper="1.570796325" velocity="100"/>
   </joint>
-  <link name="link7">
+  <link name="$(arg robot_name)_link7">
   <inertial>
           <mass value="2.24"/>
@@ -194,71 +190,71 @@
      <collision>
       <geometry>
-        <mesh filename="package://puma560_description/meshes/puma_link7.stl" scale="0.0254 0.0254 0.0254"/>
+        <box size="0.01 0.01 0.01"/>
       </geometry>
       <origin rpy="0 0 0" xyz="0 0 -0.010"/>
     </collision>
   </link>
-  <joint name="effector_revolute" type="revolute">
-    <parent link="link6"/>
-    <child link="link7"/>
+  <joint name="$(arg robot_name)_effector_revolute" type="revolute">
+    <parent link="$(arg robot_name)_link6"/>
+    <child link="$(arg robot_name)_link7"/>
     <origin rpy="-1.570796325 0 0" xyz="0 0.0558 0"/>
     <axis xyz="0 0 1"/>
     <limit effort="21.3" lower="-1.570796325" upper="1.570796325" velocity="100"/>
   </joint>
-  <ros2_control name="GazeboSystem" type="system">
+  <ros2_control name="$(arg robot_name)_GazeboSystem" type="system">
     <hardware>
       <plugin>gazebo_ros2_control/GazeboSystem</plugin>
     </hardware>
-    <joint name="platform">
-      <command_interface name="effort">
-        <param name="min">-1</param>
-        <param name="max">1</param>
-      </command_interface>
-      <state_interface name="position">
-        <param name="initial_value"></param>
-      </state_interface>
-      <state_interface name="velocity"/>
-    </joint>
-    <joint name="shoulder">
-      <command_interface name="effort">
-        <param name="min">-1</param>
-        <param name="max">1</param>
-      </command_interface>
-      <state_interface name="position">
-        <param name="initial_value"></param>
-      </state_interface>
-      <state_interface name="velocity"/>
-    </joint>
-    <joint name="elbow">
-      <command_interface name="effort">
-        <param name="min">-1</param>
-        <param name="max">1</param>
-      </command_interface>
-      <state_interface name="position">
-        <param name="initial_value"></param>
-      </state_interface>
-      <state_interface name="velocity"/>
-    </joint>
-    <joint name="wrist_revolute">
-      <command_interface name="effort">
-        <param name="min">-1</param>
-        <param name="max">1</param>
-      </command_interface>
-      <state_interface name="position">
-        <param name="initial_value"></param>
-      </state_interface>
-      <state_interface name="velocity"/>
-    </joint>
-    <joint name="wrist_bend">
-      <command_interface name="effort">
-        <param name="min">-1</param>
-        <param name="max">1</param>
-      </command_interface>
-      <state_interface name="position">
-        <param name="initial_value"></param>
-      </state_interface>
-      <state_interface name="velocity"/>
-    </joint>
-    <joint name="effector_revolute">
+    <joint name="$(arg robot_name)_platform">
+      <command_interface name="effort">
+        <param name="min">-1</param>
+        <param name="max">1</param>
+      </command_interface>
+      <state_interface name="position">
+        <param name="initial_value"></param>
+      </state_interface>
+      <state_interface name="velocity"/>
+    </joint>
+    <joint name="$(arg robot_name)_shoulder">
+      <command_interface name="effort">
+        <param name="min">-1</param>
+        <param name="max">1</param>
+      </command_interface>
+      <state_interface name="position">
+        <param name="initial_value"></param>
+      </state_interface>
+      <state_interface name="velocity"/>
+    </joint>
+    <joint name="$(arg robot_name)_elbow">
+      <command_interface name="effort">
+        <param name="min">-1</param>
+        <param name="max">1</param>
+      </command_interface>
+      <state_interface name="position">
+        <param name="initial_value"></param>
+      </state_interface>
+      <state_interface name="velocity"/>
+    </joint>
+    <joint name="$(arg robot_name)_wrist_revolute">
+      <command_interface name="effort">
+        <param name="min">-1</param>
+        <param name="max">1</param>
+      </command_interface>
+      <state_interface name="position">
+        <param name="initial_value"></param>
+      </state_interface>
+      <state_interface name="velocity"/>
+    </joint>
+    <joint name="$(arg robot_name)_wrist_bend">
+      <command_interface name="effort">
+        <param name="min">-1</param>
+        <param name="max">1</param>
+      </command_interface>
+      <state_interface name="position">
+        <param name="initial_value"></param>
+      </state_interface>
+      <state_interface name="velocity"/>
+    </joint>
+    <joint name="$(arg robot_name)_effector_revolute">
       <command_interface name="effort">
         <param name="min">-1</param>
@@ -272,8 +268,10 @@
   </ros2_control>
   <gazebo>
-    <plugin name="gazebo_ros2_control" filename="libgazebo_ros2_control.so">
-      <parameters>$(find puma560_description)/config/joint_controller.yaml</parameters>
-    </plugin>
-    <plugin name="joint_setter_plugin" filename="libjoint_setter_plugin.so">
+    <plugin name="$(arg robot_name)_gazebo_ros2_control" filename="libgazebo_ros2_control.so">
+      <ros>
+        <namespace>$(arg robot_name)</namespace>
+      </ros>
+      <parameters>$(find puma560_description)/config/$(arg robot_name)_controller.yaml</parameters>
+      <robot_param_node>/$(arg robot_name)/$(arg robot_name)_robot_state_publisher</robot_param_node>
     </plugin>
   </gazebo>
